Commit message: compiled version

File: rotors_description/urdf/multirotor_base.xacro (robot description, xacro)
@@ -132,3 +132,142 @@
     </gazebo>
   </xacro:macro>
+  <!-- Viswa's Manipulator -->
+  <!-- <link name="${namespace}/box0">
+    <xacro:box_inertial x="0.05" y="0.025" z="0.025" mass="0.001">
+      <origin xyz="0 0 0" />
+    </xacro:box_inertial>
+    <visual>
+      <origin xyz="0 0 0" rpy="0 0 0.785" />
+      <geometry>
+        <box size="0.5 0.02 0.02" />
+      </geometry>
+    </visual>
+    <collision>
+      <origin xyz="0 0 0" rpy="0 0 0.0" />
+      <geometry>
+        <box size="0.5 0.02 0.02" />
+      </geometry>
+      <surface>
+        <friction>
+          <ode>
+            <mu>5000</mu>
+            <mu2>5000</mu2>
+          </ode>
+        </friction>
+      </surface>
+    </collision>
+  </link>
+  <joint name="${namespace}/base_joint_box" type="fixed">
+    <origin xyz="0.21 0.21 0.0" rpy="0 0 0" />
+    <parent link="${namespace}/base_link" />
+    <child link="${namespace}/box0" />
+  </joint>
+  <link name="${namespace}/sensor">
+    <inertial>
+      <mass value="0.001"/>
+      <inertia ixx="0.004" ixy="0.0" ixz="0.0" iyy="0.004" iyz="0.0" izz="0.002" />
+    </inertial>
+    <visual>
+      <origin xyz="0 0 0" rpy="0 1.57 0.785" />
+      <geometry>
+        <cylinder length="0.02" radius="0.1" />
+      </geometry>
+    </visual>
+    <collision>
+      <origin xyz="0 0 0" rpy="0 1.57 0.785" />
+      <geometry>
+        <cylinder length="0.02" radius="0.1" />
+      </geometry>
+      <surface>
+        <friction>
+          <ode>
+            <mu>5000</mu>
+            <mu2>5000</mu2>
+          </ode>
+        </friction>
+      </surface>
+    </collision>
+  </link>
+  <joint name="${namespace}/base_joint_sensor" type="revolute">
+    <parent link="${namespace}/box0" />
+    <child link="${namespace}/sensor" />
+    <origin xyz="0.18 0.18 0.0" rpy="0.0 0.0 0.0" />
+    <axis xyz="1 0 0" />
+    <limit effort="10" lower="-0.1" upper="0.1" velocity="1" />
+  </joint> -->
+<!-- Achilleas' Manipulator -->
+  <!-- <link name="${namespace}/box0">
+    <inertial>
+      <mass value="0.001"/>
+      <inertia ixx="0.004" ixy="0.0" ixz="0.0" iyy="0.004" iyz="0.0" izz="0.002" />
+    </inertial>
+    <visual>
+      <origin xyz="0 0 0" rpy="0 1.57 0.785" />
+      <geometry>
+        <cylinder length="0.5" radius="0.01" />
+      </geometry>
+    </visual>
+    <collision>
+      <origin xyz="0 0 0" rpy="0 1.57 0.785" />
+      <geometry>
+        <cylinder length="0.5" radius="0.01" />
+      </geometry>
+      <surface>
+        <friction>
+          <ode>
+            <mu>5000</mu>
+            <mu2>5000</mu2>
+          </ode>
+        </friction>
+      </surface>
+    </collision>
+  </link>
+  <joint name="${namespace}/base_joint_box" type="fixed">
+    <origin xyz="0.21 0.21 0.0" rpy="0 0 0" />
+    <parent link="${namespace}/base_link" />
+    <child link="${namespace}/box0" />
+  </joint>
+  <link name="${namespace}/sensor">
+    <inertial>
+      <mass value="0.001"/>
+      <inertia ixx="0.004" ixy="0.0" ixz="0.0" iyy="0.004" iyz="0.0" izz="0.002" />
+    </inertial>
+    <visual>
+      <origin xyz="0 0 0" rpy="0 1.57 0.785" />
+      <geometry>
+        <cylinder length="0.02" radius="0.025" />
+      </geometry>
+    </visual>
+    <collision>
+      <origin xyz="0 0 0" rpy="0 1.57 0.785" />
+      <geometry>
+        <cylinder length="0.02" radius="0.025" />
+      </geometry>
+      <surface>
+        <friction>
+          <ode>
+            <mu>5000</mu>
+            <mu2>5000</mu2>
+          </ode>
+        </friction>
+      </surface>
+    </collision>
+  </link>
+  <joint name="${namespace}/box_joint_sensor" type="revolute">
+    <parent link="${namespace}/box0" />
+    <child link="${namespace}/sensor" />
+    <origin xyz="0.18 0.18 0.0" rpy="0.0 0.0 0.0" />
+    <axis xyz="1 0 0" />
+    <limit effort="10" lower="-0.1" upper="0.1" velocity="1" />
+  </joint>
+  <gazebo reference="${namespace}/box_joint_sensor">
+    <provideFeedback>true</provideFeedback>
+  </gazebo>
+  <gazebo>
+    <plugin name="ft_sensor" filename="libgazebo_ros_ft_sensor.so">
+      <updateRate>100.0</updateRate>
+      <topicName>sensor_1</topicName>
+      <jointName>${namespace}/box_joint_sensor</jointName>
+    </plugin>
+  </gazebo> -->
 </robot>

File: rotors_description/urdf/pelican.xacro (robot description, xacro)
@@ -20,4 +20,5 @@
   <!-- TODO(ff): Update these params when identifying the model. -->
   <xacro:property name="namespace" value="$(arg namespace)" />
+  <xacro:property name="color" value="$(arg color)" />
   <xacro:property name="rotor_velocity_slowdown_sim" value="10" />
   <xacro:property name="use_mesh_file" value="true" />
@@ -34,5 +35,5 @@
   <xacro:property name="time_constant_up" value="0.0125" /> <!-- [s] -->
   <xacro:property name="time_constant_down" value="0.025" /> <!-- [s] -->
-  <xacro:property name="max_rot_velocity" value="838" /> <!-- [rad/s] -->
+  <xacro:property name="max_rot_velocity" value="1838" /> <!-- [rad/s] -->
   <xacro:property name="rotor_drag_coefficient" value="8.06428e-05" />
   <xacro:property name="rolling_moment_coefficient" value="0.000001" />
@@ -142,3 +143,51 @@
     <xacro:insert_block name="rotor_inertia" />
   </xacro:vertical_rotor>
+  <!-- Macro for the inertia of a cylinder -->
+  <xacro:macro name="cyl_inertia" params="h r mass">
+    <inertia ixx="${0.0833333 * mass * (3*r*r + h*h)}" ixy="0.0" ixz="0.0"
+      iyy="${0.0833333 * mass * (3*r*r + h*h)}" iyz="0.0"
+      izz="${0.5 * mass * (r*r)}" />
+  </xacro:macro>
+<link name="${namespace}/top_rod">
+    <visual>
+      <geometry>
+        <cylinder length="0.12" radius="0.02"/>
+      </geometry>
+    </visual>
+    <collision>
+      <geometry>
+        <cylinder length="0.12" radius="0.05"/>
+      </geometry>
+    </collision>
+    <inertial>
+      <mass value="0.01"/>
+      <xacro:cyl_inertia h="0.12" r="0.05" mass="0.01"/>
+    </inertial>
+</link>
+<joint name="${namespace}/base_to_top_rod" type="fixed">
+  <origin xyz="0 0 0.12" rpy="0 0 0" />
+  <parent link="${namespace}/base_link" />
+  <child link="${namespace}/top_rod" />
+</joint>
+<link name="${namespace}/front_rod">
+    <visual>
+      <geometry>
+        <cylinder length="0.4" radius="0.01"/>
+      </geometry>
+    </visual>
+    <collision>
+      <geometry>
+        <cylinder length="0.4" radius="0.01"/>
+      </geometry>
+    </collision>
+    <inertial>
+      <mass value="0.01"/>
+      <xacro:cyl_inertia h="0.4" r="0.01" mass="0.01"/>
+    </inertial>
+</link>
+<joint name="${namespace}/top_to_front_rod" type="fixed">
+  <origin xyz="0.2 0 0.05" rpy="0 ${pi/2} 0" />
+  <parent link="${namespace}/top_rod" />
+  <child link="${namespace}/front_rod" />
+</joint>
 </robot>
